File: spring_reverb_8R_driver.brd (EAGLE design)
At the start: 100.6 x 81.3 mm, 29 parts, among them IC1 TL074P, U1 POWER

Commit message: panel
Routing:
- net +12V: track 61.4 -> 57.9 mm
- net GND: track 297.8 -> 295.4 mm
Changed lines of the file:
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@@
 <contactref element="C9" pad="2"/>
 <contactref element="C10" pad="1"/>
-<wire x1="34.925" y1="12.065" x2="35.56" y2="4.445" width="0.8128" layer="16"/>
-<wire x1="35.56" y1="4.445" x2="36.195" y2="5.715" width="0.8128" layer="16"/>
+<wire x1="34.925" y1="12.065" x2="34.925" y2="8.255" width="0.8128" layer="16"/>
+<wire x1="34.925" y1="8.255" x2="36.195" y2="5.715" width="0.8128" layer="16"/>
 <wire x1="29.845" y1="12.065" x2="34.925" y2="12.065" width="0.8128" layer="16"/>
 <wire x1="38.735" y1="5.715" x2="38.735" y2="3.175" width="0.8128" layer="16"/>
@@
 <wire x1="26.67" y1="17.145" x2="27.305" y2="12.065" width="0.8128" layer="16"/>
 <wire x1="31.115" y1="5.715" x2="31.115" y2="3.175" width="0.8128" layer="16"/>
-<wire x1="31.115" y1="5.715" x2="31.75" y2="3.81" width="0.8128" layer="16"/>
-<wire x1="27.94" y1="8.89" x2="31.75" y2="3.81" width="0.8128" layer="16"/>
-<wire x1="27.94" y1="8.89" x2="27.305" y2="12.065" width="0.8128" layer="16"/>
+<wire x1="31.115" y1="5.715" x2="31.115" y2="7.62" width="0.8128" layer="16"/>
+<wire x1="27.305" y1="10.795" x2="31.115" y2="7.62" width="0.8128" layer="16"/>
+<wire x1="27.305" y1="10.795" x2="27.305" y2="12.065" width="0.8128" layer="16"/>
 <wire x1="19.05" y1="52.705" x2="21.59" y2="48.26" width="0.8128" layer="16"/>
 <wire x1="21.59" y1="48.26" x2="24.13" y2="47.625" width="0.8128" layer="16"/>
